Commit message: Contact sensors

File: bimanual_handover/config/urdf/gen3_4f.urdf (robot description, URDF)
Before this commit: robot gen3, 32 links, 31 joints
Links:
- removed link link_0.0
- removed link link_1.0
- removed link link_10.0
- removed link link_11.0
- removed link link_11.0_tip
- removed link link_12.0
- removed link link_13.0
- removed link link_14.0
- removed link link_15.0
- removed link link_15.0_tip
- removed link link_2.0
- removed link link_3.0
- removed link link_3.0_tip
- removed link link_4.0
- removed link link_5.0
- removed link link_6.0
- removed link link_7.0
- removed link link_7.0_tip
- removed link link_8.0
- removed link link_9.0
- removed link palm_link
- added link hand_link_0.0_link, mass 0.0119; collision box size=0.0196 0.0275 0.0164; visual mesh filename=./../meshes/allegro/meshes/allegro/link_0.0.obj
- added link hand_link_1.0_link, mass 0.065; collision box size=0.0196 0.0275 0.054; visual mesh filename=./../meshes/allegro/meshes/allegro/link_1.0.obj
- added link hand_link_10._link, mass 0.0355; collision box size=0.0196 0.0275 0.0384; visual mesh filename=./../meshes/allegro/meshes/allegro/link_2.0.obj
- added link hand_link_11._link, mass 0.0096; collision sphere radius=0.0001; visual mesh filename=./../meshes/allegro/meshes/allegro/link_3.0.obj
- added link hand_link_11._link_tip_link, mass 0.0168; collision sphere radius=0.01235; visual mesh filename=./../meshes/allegro/meshes/allegro/digit.obj
- added link hand_link_12._link, mass 0.0176; collision box size=0.0358 0.034 0.0455; visual mesh filename=./../meshes/allegro/meshes/allegro/link_12.0_left.obj
- added link hand_link_13._link, mass 0.0119; collision box size=0.0196 0.0275 0.0177; visual mesh filename=./../meshes/allegro/meshes/allegro/link_13.0.obj
- added link hand_link_14._link, mass 0.038; collision box size=0.0196 0.0275 0.0514; visual mesh filename=./../meshes/allegro/meshes/allegro/link_14.0.obj
- added link hand_link_15._link, mass 0.0388; collision sphere radius=0.0001; visual mesh filename=./../meshes/allegro/meshes/allegro/link_15.0.obj
- added link hand_link_15._link_tip_link, mass 0.0168; collision sphere radius=0.01235; visual mesh filename=./../meshes/allegro/meshes/allegro/digit.obj
- added link hand_link_2.0_link, mass 0.0355; collision box size=0.0196 0.0275 0.0384; visual mesh filename=./../meshes/allegro/meshes/allegro/link_2.0.obj
- added link hand_link_3.0_link, mass 0.0096; collision sphere radius=0.0001; visual mesh filename=./../meshes/allegro/meshes/allegro/link_3.0.obj
- added link hand_link_3.0_link_tip_link, mass 0.0168; collision sphere radius=0.01235; visual mesh filename=./../meshes/allegro/meshes/allegro/digit.obj
- added link hand_link_4.0_link, mass 0.0119; collision box size=0.0196 0.0275 0.0164; visual mesh filename=./../meshes/allegro/meshes/allegro/link_0.0.obj
- added link hand_link_5.0_link, mass 0.065; collision box size=0.0196 0.0275 0.054; visual mesh filename=./../meshes/allegro/meshes/allegro/link_1.0.obj
- added link hand_link_6.0_link, mass 0.0355; collision box size=0.0196 0.0275 0.0384; visual mesh filename=./../meshes/allegro/meshes/allegro/link_2.0.obj
- added link hand_link_7.0_link, mass 0.0096; collision sphere radius=0.0001; visual mesh filename=./../meshes/allegro/meshes/allegro/link_3.0.obj
- added link hand_link_7.0_link_tip_link, mass 0.0168; collision sphere radius=0.01235; visual mesh filename=./../meshes/allegro/meshes/allegro/digit.obj
- added link hand_link_8.0_link, mass 0.0119; collision box size=0.0196 0.0275 0.0164; visual mesh filename=./../meshes/allegro/meshes/allegro/link_0.0.obj
- added link hand_link_9.0_link, mass 0.065; collision box size=0.0196 0.0275 0.054; visual mesh filename=./../meshes/allegro/meshes/allegro/link_1.0.obj
- added link hand_palm_link, mass 0.4154; collision box size=0.01 0.01 0.01; visual mesh filename=./../meshes/allegro/meshes/allegro/base_link_left.obj
Joints:
- removed joint joint_11.0_tip
- removed joint joint_15.0_tip
- removed joint joint_3.0_tip
- removed joint joint_7.0_tip
- added joint joint_11.0_tip_link: type fixed, parent hand_link_11._link, child hand_link_11._link_tip_link, origin xyz=0.02 0 0.03 rpy=0 0 0
- added joint joint_15.0_tip_link: type fixed, parent hand_link_15._link, child hand_link_15._link_tip_link, origin xyz=0.02 0 0.0455 rpy=0 0 0
- added joint joint_3.0_tip_link: type fixed, parent hand_link_3.0_link, child hand_link_3.0_link_tip_link, origin xyz=0.02 0 0.03 rpy=0 0 0
- added joint joint_7.0_tip_link: type fixed, parent hand_link_7.0_link, child hand_link_7.0_link_tip_link, origin xyz=0.02 0 0.03 rpy=0 0 0
- joint joint_0.0: child link_0.0 -> hand_link_0.0_link; parent palm_link -> hand_palm_link
- joint joint_1.0: child link_1.0 -> hand_link_1.0_link; parent link_0.0 -> hand_link_0.0_link
- joint joint_10.0: child link_10.0 -> hand_link_10._link; parent link_9.0 -> hand_link_9.0_link
- joint joint_11.0: child link_11.0 -> hand_link_11._link; parent link_10.0 -> hand_link_10._link
- joint joint_12.0: child link_12.0 -> hand_link_12._link; parent palm_link -> hand_palm_link
- joint joint_13.0: child link_13.0 -> hand_link_13._link; parent link_12.0 -> hand_link_12._link
- joint joint_14.0: child link_14.0 -> hand_link_14._link; parent link_13.0 -> hand_link_13._link
- joint joint_15.0: child link_15.0 -> hand_link_15._link; parent link_14.0 -> hand_link_14._link
- joint joint_2.0: child link_2.0 -> hand_link_2.0_link; parent link_1.0 -> hand_link_1.0_link
- joint joint_3.0: child link_3.0 -> hand_link_3.0_link; parent link_2.0 -> hand_link_2.0_link
- joint joint_4.0: child link_4.0 -> hand_link_4.0_link; parent palm_link -> hand_palm_link
- joint joint_5.0: child link_5.0 -> hand_link_5.0_link; parent link_4.0 -> hand_link_4.0_link
- joint joint_6.0: child link_6.0 -> hand_link_6.0_link; parent link_5.0 -> hand_link_5.0_link
- joint joint_7.0: child link_7.0 -> hand_link_7.0_link; parent link_6.0 -> hand_link_6.0_link
- joint joint_8.0: child link_8.0 -> hand_link_8.0_link; parent palm_link -> hand_palm_link
- joint joint_9.0: child link_9.0 -> hand_link_9.0_link; parent link_8.0 -> hand_link_8.0_link
- joint palm_2_ur: child palm_link -> hand_palm_link; origin xyz=0.0 0 0.0911750 rpy=0 0 -3.92 -> xyz=0.0 0 0.1175 rpy=0 0 5.5

File: bimanual_handover/config/urdf/ur5e_4f_ros2.urdf (robot description, URDF)
Before this commit: robot robot, 46 links, 45 joints
Links:
- removed link link_0.0
- removed link link_1.0
- removed link link_10.0
- removed link link_11.0
- removed link link_11.0_tip
- removed link link_12.0
- removed link link_13.0
- removed link link_14.0
- removed link link_15.0
- removed link link_15.0_tip
- removed link link_2.0
- removed link link_3.0
- removed link link_3.0_tip
- removed link link_4.0
- removed link link_5.0
- removed link link_6.0
- removed link link_7.0
- removed link link_7.0_tip
- removed link link_8.0
- removed link link_9.0
- removed link palm_link
- added link hand_link_0.0_link, mass 0.0119; collision box size=0.0196 0.0275 0.0164; visual mesh filename=./../meshes/allegro/meshes/allegro/link_0.0.obj
- added link hand_link_1.0_link, mass 0.065; collision box size=0.0196 0.0275 0.054; visual mesh filename=./../meshes/allegro/meshes/allegro/link_1.0.obj
- added link hand_link_10._link, mass 0.0355; collision box size=0.0196 0.0275 0.0384; visual mesh filename=./../meshes/allegro/meshes/allegro/link_2.0.obj
- added link hand_link_11._link, mass 0.0096; collision sphere radius=0.0001; visual mesh filename=./../meshes/allegro/meshes/allegro/link_3.0.obj
- added link hand_link_11._link_tip_link, mass 0.0168; collision sphere radius=0.01235; visual mesh filename=./../meshes/allegro/meshes/allegro/digit.obj
- added link hand_link_12._link, mass 0.0176; collision box size=0.0358 0.034 0.0455; visual mesh filename=./../meshes/allegro/meshes/allegro/link_12.0_left.obj
- added link hand_link_13._link, mass 0.0119; collision box size=0.0196 0.0275 0.0177; visual mesh filename=./../meshes/allegro/meshes/allegro/link_13.0.obj
- added link hand_link_14._link, mass 0.038; collision box size=0.0196 0.0275 0.0514; visual mesh filename=./../meshes/allegro/meshes/allegro/link_14.0.obj
- added link hand_link_15._link, mass 0.0388; collision sphere radius=0.0001; visual mesh filename=./../meshes/allegro/meshes/allegro/link_15.0.obj
- added link hand_link_15._link_tip_link, mass 0.0168; collision sphere radius=0.01235; visual mesh filename=./../meshes/allegro/meshes/allegro/digit.obj
- added link hand_link_2.0_link, mass 0.0355; collision box size=0.0196 0.0275 0.0384; visual mesh filename=./../meshes/allegro/meshes/allegro/link_2.0.obj
- added link hand_link_3.0_link, mass 0.0096; collision sphere radius=0.0001; visual mesh filename=./../meshes/allegro/meshes/allegro/link_3.0.obj
- added link hand_link_3.0_link_tip_link, mass 0.0168; collision sphere radius=0.01235; visual mesh filename=./../meshes/allegro/meshes/allegro/digit.obj
- added link hand_link_4.0_link, mass 0.0119; collision box size=0.0196 0.0275 0.0164; visual mesh filename=./../meshes/allegro/meshes/allegro/link_0.0.obj
- added link hand_link_5.0_link, mass 0.065; collision box size=0.0196 0.0275 0.054; visual mesh filename=./../meshes/allegro/meshes/allegro/link_1.0.obj
- added link hand_link_6.0_link, mass 0.0355; collision box size=0.0196 0.0275 0.0384; visual mesh filename=./../meshes/allegro/meshes/allegro/link_2.0.obj
- added link hand_link_7.0_link, mass 0.0096; collision sphere radius=0.0001; visual mesh filename=./../meshes/allegro/meshes/allegro/link_3.0.obj
- added link hand_link_7.0_link_tip_link, mass 0.0168; collision sphere radius=0.01235; visual mesh filename=./../meshes/allegro/meshes/allegro/digit.obj
- added link hand_link_8.0_link, mass 0.0119; collision box size=0.0196 0.0275 0.0164; visual mesh filename=./../meshes/allegro/meshes/allegro/link_0.0.obj
- added link hand_link_9.0_link, mass 0.065; collision box size=0.0196 0.0275 0.054; visual mesh filename=./../meshes/allegro/meshes/allegro/link_1.0.obj
- added link hand_palm_link, mass 0.4154; collision box size=0.01 0.01 0.01; visual mesh filename=./../meshes/allegro/meshes/allegro/base_link_left.obj
Joints:
- removed joint joint_11.0_tip
- removed joint joint_15.0_tip
- removed joint joint_3.0_tip
- removed joint joint_7.0_tip
- added joint joint_11.0_tip_link: type fixed, parent hand_link_11._link, child hand_link_11._link_tip_link, origin xyz=0.02 0 0.03 rpy=0 0 0
- added joint joint_15.0_tip_link: type fixed, parent hand_link_15._link, child hand_link_15._link_tip_link, origin xyz=0.02 0 0.0455 rpy=0 0 0
- added joint joint_3.0_tip_link: type fixed, parent hand_link_3.0_link, child hand_link_3.0_link_tip_link, origin xyz=0.02 0 0.03 rpy=0 0 0
- added joint joint_7.0_tip_link: type fixed, parent hand_link_7.0_link, child hand_link_7.0_link_tip_link, origin xyz=0.02 0 0.03 rpy=0 0 0
- joint joint_0.0: child link_0.0 -> hand_link_0.0_link; parent palm_link -> hand_palm_link
- joint joint_1.0: child link_1.0 -> hand_link_1.0_link; parent link_0.0 -> hand_link_0.0_link
- joint joint_10.0: child link_10.0 -> hand_link_10._link; parent link_9.0 -> hand_link_9.0_link
- joint joint_11.0: child link_11.0 -> hand_link_11._link; parent link_10.0 -> hand_link_10._link
- joint joint_12.0: child link_12.0 -> hand_link_12._link; parent palm_link -> hand_palm_link
- joint joint_13.0: child link_13.0 -> hand_link_13._link; parent link_12.0 -> hand_link_12._link
- joint joint_14.0: child link_14.0 -> hand_link_14._link; parent link_13.0 -> hand_link_13._link
- joint joint_15.0: child link_15.0 -> hand_link_15._link; parent link_14.0 -> hand_link_14._link
- joint joint_2.0: child link_2.0 -> hand_link_2.0_link; parent link_1.0 -> hand_link_1.0_link
- joint joint_3.0: child link_3.0 -> hand_link_3.0_link; parent link_2.0 -> hand_link_2.0_link
- joint joint_4.0: child link_4.0 -> hand_link_4.0_link; parent palm_link -> hand_palm_link
- joint joint_5.0: child link_5.0 -> hand_link_5.0_link; parent link_4.0 -> hand_link_4.0_link
- joint joint_6.0: child link_6.0 -> hand_link_6.0_link; parent link_5.0 -> hand_link_5.0_link
- joint joint_7.0: child link_7.0 -> hand_link_7.0_link; parent link_6.0 -> hand_link_6.0_link
- joint joint_8.0: child link_8.0 -> hand_link_8.0_link; parent palm_link -> hand_palm_link
- joint joint_9.0: child link_9.0 -> hand_link_9.0_link; parent link_8.0 -> hand_link_8.0_link
- joint palm_2_ur: child palm_link -> hand_palm_link

Commit message: Fix: stiffness and damping of the hand joints.

File: bimanual_handover/config/urdf/gen3_4f.urdf (robot description, URDF)
Before this commit: robot gen3, 32 links, 31 joints
Joints:
- removed joint joint_1
- removed joint joint_2
- removed joint joint_3
- removed joint joint_4
- removed joint joint_5
- removed joint joint_6
- removed joint joint_7
- added joint arm_joint_1: type continuous, parent base_link, child shoulder_link, origin xyz=0 0 0.15643 rpy=3.1416 2.7629E-18 -4.9305E-36, axis 0 0 1, limit effort=39 velocity=1.3963
- added joint arm_joint_2: type revolute, parent shoulder_link, child half_arm_1_link, origin xyz=0 0.005375 -0.12838 rpy=1.5708 2.1343E-17 -1.1102E-16, axis 0 0 1, limit lower=-2.24 upper=2.24 effort=39 velocity=1.3963
- added joint arm_joint_3: type continuous, parent half_arm_1_link, child half_arm_2_link, origin xyz=0 -0.21038 -0.006375 rpy=-1.5708 1.2326E-32 -2.9122E-16, axis 0 0 1, limit effort=39 velocity=1.3963
- added joint arm_joint_4: type revolute, parent half_arm_2_link, child forearm_link, origin xyz=0 0.006375 -0.21038 rpy=1.5708 -6.6954E-17 -1.6653E-16, axis 0 0 1, limit lower=-2.57 upper=2.57 effort=39 velocity=1.3963
- added joint arm_joint_5: type continuous, parent forearm_link, child spherical_wrist_1_link, origin xyz=0 -0.20843 -0.006375 rpy=-1.5708 2.2204E-16 -6.373E-17, axis 0 0 1, limit effort=9 velocity=1.2218
- added joint arm_joint_6: type revolute, parent spherical_wrist_1_link, child spherical_wrist_2_link, origin xyz=0 0.00017505 -0.10593 rpy=1.5708 9.2076E-28 -8.2157E-15, axis 0 0 1, limit lower=-2.09 upper=2.09 effort=9 velocity=1.2218
- added joint arm_joint_7: type continuous, parent spherical_wrist_2_link, child bracelet_link, origin xyz=0 -0.10593 -0.00017505 rpy=-1.5708 -5.5511E-17 9.6396E-17, axis 0 0 1, limit effort=9 velocity=1.2218

File: bimanual_handover/config/urdf/ur5e_4f_ros2.urdf (robot description, URDF)
Before this commit: robot robot, 46 links, 45 joints
Joints:
- removed joint elbow_joint
- removed joint shoulder_lift_joint
- removed joint shoulder_pan_joint
- removed joint wrist_1_joint
- removed joint wrist_2_joint
- removed joint wrist_3_joint
- added joint arm_elbow_joint: type revolute, parent upper_arm_link, child forearm_link, origin xyz=-0.425 0 0 rpy=0 0 0, axis 0 0 1, limit lower=-3.141592653589793 upper=3.141592653589793 effort=150.0 velocity=3.141592653589793
- added joint arm_shoulder_lift_joint: type revolute, parent shoulder_link, child upper_arm_link, origin xyz=0 0 0 rpy=1.570796327 0 0, axis 0 0 1, limit lower=-6.283185307179586 upper=6.283185307179586 effort=150.0 velocity=3.141592653589793
- added joint arm_shoulder_pan_joint: type revolute, parent base_link_inertia, child shoulder_link, origin xyz=0 0 0.1625 rpy=0 0 0, axis 0 0 1, limit lower=-6.283185307179586 upper=6.283185307179586 effort=150.0 velocity=3.141592653589793
- added joint arm_wrist_1_joint: type revolute, parent forearm_link, child wrist_1_link, origin xyz=-0.3922 0 0.1333 rpy=0 0 0, axis 0 0 1, limit lower=-6.283185307179586 upper=6.283185307179586 effort=28.0 velocity=3.141592653589793
- added joint arm_wrist_2_joint: type revolute, parent wrist_1_link, child wrist_2_link, origin xyz=0 -0.0997 -2.044881182297852e-11 rpy=1.570796327 0 0, axis 0 0 1, limit lower=-6.283185307179586 upper=6.283185307179586 effort=28.0 velocity=3.141592653589793
- added joint arm_wrist_3_joint: type continuous, parent wrist_2_link, child wrist_3_link, origin xyz=0 0.0996 -2.042830148012698e-11 rpy=1.570796326589793 3.141592653589793 3.141592653589793, axis 0 0 1, limit effort=28.0 velocity=3.141592653589793

Commit message: Add: dummy links to hand fingers (inner)

File: bimanual_handover/config/urdf/gen3_4f.urdf (robot description, URDF)
Before this commit: robot gen3, 32 links, 31 joints
Links:
- added link finger_1_contact_1; collision box size=0.00125 0.017 0.065; visual box size=0.00125 0.017 0.065
- added link finger_1_contact_2; collision box size=0.00125 0.017 0.0375; visual box size=0.00125 0.017 0.0375
- added link finger_1_contact_3_tip; collision box size=0.00075 0.02 0.02; visual box size=0.00075 0.02 0.02
- added link finger_2_contact_5; collision box size=0.00125 0.017 0.065; visual box size=0.00125 0.017 0.065
- added link finger_2_contact_6; collision box size=0.00125 0.017 0.0375; visual box size=0.00125 0.017 0.0375
- added link finger_2_contact_7_tip; collision box size=0.00075 0.02 0.02; visual box size=0.00075 0.02 0.02
- added link finger_3_contact_10; collision box size=0.00125 0.017 0.0375; visual box size=0.00125 0.017 0.0375
- added link finger_3_contact_11_tip; collision box size=0.00075 0.02 0.02; visual box size=0.00075 0.02 0.02
- added link finger_3_contact_9; collision box size=0.00125 0.017 0.065; visual box size=0.00125 0.017 0.065
- added link finger_4_contact_14; collision box size=0.00125 0.022 0.0375; visual box size=0.00125 0.022 0.0375
- added link finger_4_contact_15; collision box size=0.00125 0.022 0.035; visual box size=0.00125 0.022 0.035
- added link finger_4_contact_15_tip; collision box size=0.00075 0.02 0.02; visual box size=0.00075 0.02 0.02
Joints:
- added joint finger_1_contact2_1: type fixed, parent hand_link_1.0_link, child finger_1_contact_1, origin xyz=0.01 0 0.0275 rpy=0 0 0
- added joint finger_1_contact2_2: type fixed, parent hand_link_2.0_link, child finger_1_contact_2, origin xyz=0.01 0 0.0325 rpy=0 0 0
- added joint finger_1_contact2_3_tip: type fixed, parent hand_link_3.0_link_tip_link, child finger_1_contact_3_tip, origin xyz=0 0 0 rpy=0 0 0
- added joint finger_2_contact2_7_tip: type fixed, parent hand_link_7.0_link_tip_link, child finger_2_contact_7_tip, origin xyz=0 0 0 rpy=0 0 0
- added joint finger_2_contact5_1: type fixed, parent hand_link_5.0_link, child finger_2_contact_5, origin xyz=0.01 0 0.0275 rpy=0 0 0
- added joint finger_2_contact6_2: type fixed, parent hand_link_6.0_link, child finger_2_contact_6, origin xyz=0.01 0 0.0325 rpy=0 0 0
- added joint finger_3_contact10_2: type fixed, parent hand_link_10._link, child finger_3_contact_10, origin xyz=0.01 0 0.0325 rpy=0 0 0
- added joint finger_3_contact2_11_tip: type fixed, parent hand_link_11._link_tip_link, child finger_3_contact_11_tip, origin xyz=0 0 0 rpy=0 0 0
- added joint finger_3_contact9_1: type fixed, parent hand_link_9.0_link, child finger_3_contact_9, origin xyz=0.01 0 0.0275 rpy=0 0 0
- added joint finger_4_contact2_14: type fixed, parent hand_link_14._link, child finger_4_contact_14, origin xyz=0.01 0 0.005 rpy=0 0 0
- added joint finger_4_contact2_15: type fixed, parent hand_link_15._link, child finger_4_contact_15, origin xyz=0.01 0 0.005 rpy=0 0 0
- added joint finger_4_contact2_15_tip: type fixed, parent hand_link_15._link_tip_link, child finger_4_contact_15_tip, origin xyz=0.0 0 0.0 rpy=0 0 0

File: bimanual_handover/config/urdf/ur5e_4f_ros2.urdf (robot description, URDF)
Before this commit: robot robot, 46 links, 45 joints
Links:
- added link finger_1_contact_1; collision box size=0.00125 0.017 0.065; visual box size=0.00125 0.017 0.065
- added link finger_1_contact_2; collision box size=0.00125 0.017 0.0375; visual box size=0.00125 0.017 0.0375
- added link finger_1_contact_3_tip; collision box size=0.00075 0.02 0.02; visual box size=0.00075 0.02 0.02
- added link finger_2_contact_5; collision box size=0.00125 0.017 0.065; visual box size=0.00125 0.017 0.065
- added link finger_2_contact_6; collision box size=0.00125 0.017 0.0375; visual box size=0.00125 0.017 0.0375
- added link finger_2_contact_7_tip; collision box size=0.00075 0.02 0.02; visual box size=0.00075 0.02 0.02
- added link finger_3_contact_10; collision box size=0.00125 0.017 0.0375; visual box size=0.00125 0.017 0.0375
- added link finger_3_contact_11_tip; collision box size=0.00075 0.02 0.02; visual box size=0.00075 0.02 0.02
- added link finger_3_contact_9; collision box size=0.00125 0.017 0.065; visual box size=0.00125 0.017 0.065
- added link finger_4_contact_14; collision box size=0.00125 0.022 0.0375; visual box size=0.00125 0.022 0.0375
- added link finger_4_contact_15; collision box size=0.00125 0.022 0.035; visual box size=0.00125 0.022 0.035
- added link finger_4_contact_15_tip; collision box size=0.00075 0.02 0.02; visual box size=0.00075 0.02 0.02
Joints:
- added joint finger_1_contact2_1: type fixed, parent hand_link_1.0_link, child finger_1_contact_1, origin xyz=0.01 0 0.0275 rpy=0 0 0
- added joint finger_1_contact2_2: type fixed, parent hand_link_2.0_link, child finger_1_contact_2, origin xyz=0.01 0 0.0325 rpy=0 0 0
- added joint finger_1_contact2_3_tip: type fixed, parent hand_link_3.0_link_tip_link, child finger_1_contact_3_tip, origin xyz=0 0 0 rpy=0 0 0
- added joint finger_2_contact2_7_tip: type fixed, parent hand_link_7.0_link_tip_link, child finger_2_contact_7_tip, origin xyz=0 0 0 rpy=0 0 0
- added joint finger_2_contact5_1: type fixed, parent hand_link_5.0_link, child finger_2_contact_5, origin xyz=0.01 0 0.0275 rpy=0 0 0
- added joint finger_2_contact6_2: type fixed, parent hand_link_6.0_link, child finger_2_contact_6, origin xyz=0.01 0 0.0325 rpy=0 0 0
- added joint finger_3_contact10_2: type fixed, parent hand_link_10._link, child finger_3_contact_10, origin xyz=0.01 0 0.0325 rpy=0 0 0
- added joint finger_3_contact2_11_tip: type fixed, parent hand_link_11._link_tip_link, child finger_3_contact_11_tip, origin xyz=0 0 0 rpy=0 0 0
- added joint finger_3_contact9_1: type fixed, parent hand_link_9.0_link, child finger_3_contact_9, origin xyz=0.01 0 0.0275 rpy=0 0 0
- added joint finger_4_contact2_14: type fixed, parent hand_link_14._link, child finger_4_contact_14, origin xyz=0.01 0 0.005 rpy=0 0 0
- added joint finger_4_contact2_15: type fixed, parent hand_link_15._link, child finger_4_contact_15, origin xyz=0.01 0 0.005 rpy=0 0 0
- added joint finger_4_contact2_15_tip: type fixed, parent hand_link_15._link_tip_link, child finger_4_contact_15_tip, origin xyz=0.0 0 0.0 rpy=0 0 0

Commit message: Add: dummy link for collision detecion in palm link

File: bimanual_handover/config/urdf/gen3_4f.urdf (robot description, URDF)
Before this commit: robot gen3, 44 links, 43 joints
Links:
- added link palm_aux_link; collision box size=0.00125 0.055 0.075; visual box size=0.00125 0.055 0.075
- added link palm_aux_link2; collision box size=0.00125 0.017 0.065; visual box size=0.00125 0.075 0.035
Joints:
- added joint palm_aux_joint: type fixed, parent hand_palm_link, child palm_aux_link, origin xyz=0.0125 0.02 -0.04 rpy=0 0 0
- added joint palm_aux_joint2: type fixed, parent hand_palm_link, child palm_aux_link2, origin xyz=0.0125 -0.02 -0.02 rpy=0 0 0
