Commit message: Modified: suffix "_link" for contacts

File: bimanual_handover/config/urdf/gen3_4f.urdf (robot description, URDF)
Before this commit: robot gen3, 46 links, 45 joints
Links:
- removed link finger_1_contact_1
- removed link finger_1_contact_2
- removed link finger_1_contact_3_tip
- removed link finger_2_contact_5
- removed link finger_2_contact_6
- removed link finger_2_contact_7_tip
- removed link finger_3_contact_10
- removed link finger_3_contact_11_tip
- removed link finger_3_contact_9
- removed link finger_4_contact_14
- removed link finger_4_contact_15
- removed link finger_4_contact_15_tip
- removed link palm_aux_link2
- added link finger_1_contact_1_link; collision box size=0.00125 0.017 0.065; visual box size=0.00125 0.017 0.065
- added link finger_1_contact_2_link; collision box size=0.00125 0.017 0.0375; visual box size=0.00125 0.017 0.0375
- added link finger_1_contact_3_tip_link; collision box size=0.00075 0.02 0.02; visual box size=0.00075 0.02 0.02
- added link finger_2_contact_5_link; collision box size=0.00125 0.017 0.065; visual box size=0.00125 0.017 0.065
- added link finger_2_contact_6_link; collision box size=0.00125 0.017 0.0375; visual box size=0.00125 0.017 0.0375
- added link finger_2_contact_7_tip_link; collision box size=0.00075 0.02 0.02; visual box size=0.00075 0.02 0.02
- added link finger_3_contact_10_link; collision box size=0.00125 0.017 0.0375; visual box size=0.00125 0.017 0.0375
- added link finger_3_contact_11_tip_link; collision box size=0.00075 0.02 0.02; visual box size=0.00075 0.02 0.02
- added link finger_3_contact_9_link; collision box size=0.00125 0.017 0.065; visual box size=0.00125 0.017 0.065
- added link finger_4_contact_14_link; collision box size=0.00125 0.022 0.0375; visual box size=0.00125 0.022 0.0375
- added link finger_4_contact_15_link; collision box size=0.00125 0.022 0.035; visual box size=0.00125 0.022 0.035
- added link finger_4_contact_15_tip_link; collision box size=0.00075 0.02 0.02; visual box size=0.00075 0.02 0.02
- added link palm_aux2_link; collision box size=0.00125 0.017 0.065; visual box size=0.00125 0.075 0.035
Joints:
- joint finger_1_contact2_1: child finger_1_contact_1 -> finger_1_contact_1_link
- joint finger_1_contact2_2: child finger_1_contact_2 -> finger_1_contact_2_link
- joint finger_1_contact2_3_tip: child finger_1_contact_3_tip -> finger_1_contact_3_tip_link
- joint finger_2_contact2_7_tip: child finger_2_contact_7_tip -> finger_2_contact_7_tip_link
- joint finger_2_contact5_1: child finger_2_contact_5 -> finger_2_contact_5_link
- joint finger_2_contact6_2: child finger_2_contact_6 -> finger_2_contact_6_link
- joint finger_3_contact10_2: child finger_3_contact_10 -> finger_3_contact_10_link
- joint finger_3_contact2_11_tip: child finger_3_contact_11_tip -> finger_3_contact_11_tip_link
- joint finger_3_contact9_1: child finger_3_contact_9 -> finger_3_contact_9_link
- joint finger_4_contact2_14: child finger_4_contact_14 -> finger_4_contact_14_link
- joint finger_4_contact2_15: child finger_4_contact_15 -> finger_4_contact_15_link
- joint finger_4_contact2_15_tip: child finger_4_contact_15_tip -> finger_4_contact_15_tip_link
- joint palm_aux_joint2: child palm_aux_link2 -> palm_aux2_link

Commit message: Modified: augment joint limit for thumb

File: bimanual_handover/config/urdf/gen3_4f.urdf (robot description, URDF)
Before this commit: robot gen3, 46 links, 45 joints
Joints:
- joint joint_13.0: limit lower=-0.105 upper=1.163 effort=0.35 velocity=6.283 -> lower=-1.05 upper=1.163 effort=0.35 velocity=6.283

Commit message: Modified: GEN3 hand joint limits increased

File: bimanual_handover/config/urdf/gen3_4f.urdf (robot description, URDF)
Before this commit: robot gen3, 46 links, 45 joints
Joints:
- joint joint_10.0: limit lower=-0.174 upper=1.709 effort=0.35 velocity=6.283 -> lower=-0.174 upper=1.4 effort=0.35 velocity=6.283
- joint joint_11.0: limit lower=-0.227 upper=1.618 effort=0.35 velocity=6.283 -> lower=-0.227 upper=1 effort=0.35 velocity=6.283
- joint joint_12.0: limit lower=0.263 upper=1.396 effort=0.35 velocity=6.283 -> lower=0.263 upper=0.7 effort=0.35 velocity=6.283
- joint joint_13.0: limit lower=-1.05 upper=1.163 effort=0.35 velocity=6.283 -> lower=-1.05 upper=0.7 effort=0.35 velocity=6.283
- joint joint_14.0: limit lower=-0.189 upper=1.644 effort=0.35 velocity=6.283 -> lower=-0.189 upper=0.8 effort=0.35 velocity=6.283
- joint joint_2.0: limit lower=-0.174 upper=1.709 effort=0.35 velocity=6.283 -> lower=-0.174 upper=1.4 effort=0.35 velocity=6.283
- joint joint_3.0: limit lower=-0.227 upper=1.618 effort=0.35 velocity=6.283 -> lower=-0.227 upper=1.0 effort=0.35 velocity=6.283
- joint joint_6.0: limit lower=-0.174 upper=1.709 effort=0.35 velocity=6.283 -> lower=-0.174 upper=1.4 effort=0.35 velocity=6.283
- joint joint_7.0: limit lower=-0.227 upper=1.618 effort=0.35 velocity=6.283 -> lower=-0.227 upper=1. effort=0.35 velocity=6.283
