Commit message: Updated: RL manipulation for reach

File: rl_manipulation/config/urdf/ur5e_ros2.urdf (robot description, URDF)
Before this commit: robot robot, 39 links, 38 joints
Links:
- removed link robotiq_finger_1_link_0
- removed link robotiq_finger_1_link_1
- removed link robotiq_finger_1_link_2
- removed link robotiq_finger_1_link_3
- removed link robotiq_finger_2_link_0
- removed link robotiq_finger_2_link_1
- removed link robotiq_finger_2_link_2
- removed link robotiq_finger_2_link_3
- removed link robotiq_finger_middle_link_0
- removed link robotiq_finger_middle_link_1
- removed link robotiq_finger_middle_link_2
- removed link robotiq_finger_middle_link_3
- removed link robotiq_palm
- removed link robotiq_tool0
Joints:
- removed joint robotiq_finger_1_joint_1
- removed joint robotiq_finger_1_joint_2
- removed joint robotiq_finger_1_joint_3
- removed joint robotiq_finger_2_joint_1
- removed joint robotiq_finger_2_joint_2
- removed joint robotiq_finger_2_joint_3
- removed joint robotiq_finger_middle_joint_1
- removed joint robotiq_finger_middle_joint_2
- removed joint robotiq_finger_middle_joint_3
- removed joint robotiq_palm_finger_1_joint
- removed joint robotiq_palm_finger_2_joint
- removed joint robotiq_palm_finger_middle_joint
- removed joint robotiq_palm_tool0
- removed joint urGripper_gripper_joint
