Commit message: Modified: wrist 3 joint as a revolute joint

File: rl_manipulation/config/urdf/ur5e_position_ros2_3f.urdf (robot description, URDF)
Before this commit: robot robot, 37 links, 36 joints
Joints:
- joint wrist_3_joint: type continuous -> revolute

Commit message: Modified: URDF without the contact in the tip

File: rl_manipulation/config/urdf/ur5e_position_ros2_3f.urdf (robot description, URDF)
Before this commit: robot robot, 37 links, 36 joints
Links:
- removed link robotiq_finger_1_contact_tip
- removed link robotiq_finger_2_contact_tip
- removed link robotiq_finger_middle_contact_tip
Joints:
- removed joint robotiq_1_contact_tip_joint
- removed joint robotiq_2_contact_tip_joint
- removed joint robotiq_middle_contact_tip_joint

Commit message: Modified: add tip contact

File: rl_manipulation/config/urdf/ur5e_position_ros2_3f.urdf (robot description, URDF)
Before this commit: robot robot, 34 links, 33 joints
Links:
- added link robotiq_finger_1_contact_tip; collision box size=0.0535 0.001 0.0235; visual box size=0.0535 0.001 0.0235
- added link robotiq_finger_2_contact_tip; collision box size=0.0535 0.001 0.0235; visual box size=0.0535 0.001 0.0235
- added link robotiq_finger_middle_contact_tip; collision box size=0.0535 0.001 0.0235; visual box size=0.0535 0.001 0.0235
Joints:
- added joint robotiq_1_contact_tip_joint: type fixed, parent robotiq_finger_1_link_3, child robotiq_finger_1_contact_tip, origin xyz=0.005 0.012 0.0 rpy=0 0 0.55
- added joint robotiq_2_contact_tip_joint: type fixed, parent robotiq_finger_2_link_3, child robotiq_finger_2_contact_tip, origin xyz=0.005 0.012 0.0 rpy=0 0 0.55
- added joint robotiq_middle_contact_tip_joint: type fixed, parent robotiq_finger_middle_link_3, child robotiq_finger_middle_contact_tip, origin xyz=0.005 0.012 0.0 rpy=0 0 0.55

Commit message: Modified: remove contact collision

File: rl_manipulation/config/urdf/ur5e_position_ros2_3f.urdf (robot description, URDF)
Before this commit: robot robot, 37 links, 36 joints
Links:
- link robotiq_finger_2_contact_2: geometry visual box size=0.05 0.0002 0.0275
- link robotiq_finger_2_contact_3: geometry visual box size=0.05 0.0002 0.0275
- link robotiq_finger_2_contact_tip: geometry visual box size=0.0535 0.001 0.0235

Commit message: Modified: USD without contact collision

File: rl_manipulation/config/urdf/ur5e_position_ros2_3f.urdf (robot description, URDF)
Before this commit: robot robot, 37 links, 36 joints
Links:
- link robotiq_finger_1_contact_2: geometry visual box size=0.05 0.0002 0.0275
- link robotiq_finger_1_contact_3: geometry visual box size=0.05 0.0002 0.0275
- link robotiq_finger_1_contact_tip: geometry visual box size=0.0535 0.001 0.0235
- link robotiq_finger_middle_contact_2: geometry visual box size=0.05 0.0002 0.0275
- link robotiq_finger_middle_contact_3: geometry visual box size=0.05 0.0002 0.0275
- link robotiq_finger_middle_contact_tip: geometry visual box size=0.0535 0.001 0.0235

Commit message: Modified: no contacts in USD

File: rl_manipulation/config/urdf/ur5e_position_ros2_3f.urdf (robot description, URDF)
Before this commit: robot robot, 37 links, 36 joints
Links:
- removed link robotiq_finger_1_contact_2
- removed link robotiq_finger_1_contact_3
- removed link robotiq_finger_1_contact_tip
- removed link robotiq_finger_2_contact_2
- removed link robotiq_finger_2_contact_3
- removed link robotiq_finger_2_contact_tip
- removed link robotiq_finger_middle_contact_2
- removed link robotiq_finger_middle_contact_3
- removed link robotiq_finger_middle_contact_tip
Joints:
- removed joint robotiq_1_contact_2_joint
- removed joint robotiq_1_contact_3_joint
- removed joint robotiq_1_contact_tip_joint
- removed joint robotiq_2_contact_2_joint
- removed joint robotiq_2_contact_3_joint
- removed joint robotiq_2_contact_tip_joint
- removed joint robotiq_middle_contact_2_joint
- removed joint robotiq_middle_contact_3_joint
- removed joint robotiq_middle_contact_tip_joint
